File: ESP-IP.kicad_sch (KiCad schematic)
At the start: 32 parts, among them J1 Serial and power, J2 Programming Pads, Q1 L78M05ABDT-TR, SW1 SW_Push, SW2 SW_Push, U1 ESP32-WROOM-32U, U3 TXS0102DCU, U4 AMS1117-3.3

Commit message: feat: moving around bits and bobs
Parts:
- R1: footprint LED_SMD:LED_0402_1005Metric -> Resistor_SMD:R_0805_2012Metric
Changed lines of the file:
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@@
       (effects (font (size 1.27 1.27)))
     )
-    (property "Footprint" "LED_SMD:LED_0402_1005Metric" (at 253.365 84.328 90)
+    (property "Footprint" "Resistor_SMD:R_0805_2012Metric" (at 253.365 84.328 90)
       (effects (font (size 1.27 1.27)) hide)
     )
